File: 238S.sch (KiCad schematic (older format))
At the start: 75 parts, among them J1 Conn_01x09, J2 Conn_01x14, Q30 Q_PNP_EBC, Q31 Q_NPN_EBC, Q4 Q_NPN_EBC, U13 DTA124E, U14 DTA124E, U15 DTA124E, U16 DTA124E, U17 DTC124E, U20 uPC4570HA, U30 TEACDOLBYS, U31 NJM4560, U4 4066, U8 uPC4570HA

Commit message: Add values
Parts:
- C34, C36, C37, C38, C52, C54, C80, C84: value CP1 -> 10/16
- C35: value C -> 470p
- C51: value C -> 100p
- C81, C83, C85: value CP1 -> 4.7/50
- C82: value CP1 -> 2.2/50
- C86, C87: value CP1 -> 47/16
- Q30: value Q_PNP_EBC -> PNP
- Q31: value Q_NPN_EBC -> NPN
- Q4: value Q_NPN_EBC -> 2SD1450
- R22, R23, R24, R39, R41, R46, R65, R66, R72: value R_US -> 10k
- R25, R89, R92: value R_US -> 220k
- R33, R73: value R_US -> 47k
- R34, R37, R43: value R_US -> 100k
- R35: value R_US -> 3k
- R36: value R_US -> 1.2k
- R38: value R_US -> 22k
- R40, R75: value R_US -> 68k
- R47, R91: value R_POT_US -> 47k
- R64, R80, R87: value R_US -> 4.7k
- R70: value R_US -> 470
- R71: value R_US -> 24k
- R74: value R_US -> 1.5k
- R81: value R_US -> 3.3k
- R82, R88, R94: value R_POT_US -> 4.7k
- R83, R85: value R_US -> 1k
- R84, R93: value R_US -> 2.2k
- R86: value R_US -> 15k
- R90: value R_US -> 82k
- U30: value TEACDOLBYS -> TEAC_DOLBY_S_CARD
- U31: value NJM4560 -> NJM4565
Connections:
- net FROM_PLAY_AMP renamed PLAY_AMP_OUTPUT
- net TO_REC_AMP renamed REC_AMP_INPUT
Other:
- note added: "Tascam 238S R/P AMP PCB\nCircuits specific to Dolby S\nPlayback amp, record amp and erase circuits are identical to 238\n238pro.com\nv2020.10.10"
- note removed: "Tascam 238S R/P AMP PCB Dolby S specific circuits"
- moved on the sheet: C87, J2

Commit message: Latest schematics
Parts:
- removed Q30: PNP, symbol Device:Q_PNP_EBC
- removed Q31: NPN, symbol Device:Q_NPN_EBC
- added Q30: J4021D, symbol Device:Q_PJFET_DGS
- added Q31: K8124D, symbol Device:Q_NJFET_DGS
Other:
- note added: "Tascam 238S R/P AMP PCB\nCircuits specific to Dolby S\nPlayback amp, record amp and erase circuits are identical to 238\n238pro.com\nv2020.10.27"
- note removed: "Tascam 238S R/P AMP PCB\nCircuits specific to Dolby S\nPlayback amp, record amp and erase circuits are identical to 238\n238pro.com\nv2020.10.10"
Changed lines of the file:
@@
 $Descr USLetter 11000 8500
 encoding utf-8
-Sheet 1 2
+Sheet 1 1
 Title ""
 Date ""
@@
 Wire Wire Line
 	2100 4500 2100 4650
-$Comp
-L Device:Q_PNP_EBC Q30
-U 1 1 5F807F96
-P 6550 1300
-F 0 "Q30" H 6740 1254 50  0000 L CNN
-F 1 "PNP" H 6740 1345 50  0000 L CNN
-F 2 "" H 6750 1400 50  0001 C CNN
-F 3 "~" H 6550 1300 50  0001 C CNN
-	1    6550 1300
-	1    0    0    1
-$EndComp
 Wire Wire Line
 	4100 950  6650 950
@@
 	1    6200 1300
 	-1   0    0    1
-$EndComp
-$Comp
-L Device:Q_NPN_EBC Q31
-U 1 1 5F80BFEA
-P 6550 2150
-F 0 "Q31" H 6741 2104 50  0000 L CNN
-F 1 "NPN" H 6741 2195 50  0000 L CNN
-F 2 "" H 6750 2250 50  0001 C CNN
-F 3 "~" H 6550 2150 50  0001 C CNN
-	1    6550 2150
-	1    0    0    1
 $EndComp
 Wire Wire Line
@@
 	5600 2500 6050 2500
 Text Notes 750  7950 0    79   ~ 0
-Tascam 238S R/P AMP PCB\nCircuits specific to Dolby S\nPlayback amp, record amp and erase circuits are identical to 238\n238pro.com\nv2020.10.10
-$Sheet
-S 11350 6400 4000 800
-U 5F8BA977
-F0 "DolbyS-NR-HIC" 50
-F1 "DolbyS-NR-HIC.sch" 50
-$EndSheet
+Tascam 238S R/P AMP PCB\nCircuits specific to Dolby S\nPlayback amp, record amp and erase circuits are identical to 238\n238pro.com\nv2020.10.27
+$Comp
+L Device:Q_NJFET_DGS Q31
+U 1 1 5F96A47F
+P 6550 2150
+F 0 "Q31" H 6740 2104 50  0000 L CNN
+F 1 "K8124D" H 6740 2195 50  0000 L CNN
+F 2 "" H 6750 2250 50  0001 C CNN
+F 3 "~" H 6550 2150 50  0001 C CNN
+	1    6550 2150
+	1    0    0    1
+$EndComp
+$Comp
+L Device:Q_PJFET_DGS Q30
+U 1 1 5F96BCED
+P 6550 1300
+F 0 "Q30" H 6741 1254 50  0000 L CNN
+F 1 "J4021D" H 6741 1345 50  0000 L CNN
+F 2 "" H 6750 1400 50  0001 C CNN
+F 3 "~" H 6550 1300 50  0001 C CNN
+	1    6550 1300
+	1    0    0    1
+$EndComp
 $EndSCHEMATC
